Commit message: feat: add calibrated direct Cartesian grasping

File: simulation/urdf/mycobot_description/urdf/mecharm_270_pi/mecharm_270_pi_adaptive_gripper.urdf (robot description, URDF)
Before this commit: robot firefighter, 14 links, 13 joints
Links:
- added link gripper_tcp
Joints:
- added joint gripper_base_to_tcp: type fixed, parent gripper_base, child gripper_tcp, origin xyz=0 0.034 0 rpy=0 0 0

Commit message: fix: stabilize adaptive gripper loop physics and refresh scene

File: simulation/urdf/mycobot_description/urdf/mecharm_270_pi/mecharm_270_pi_adaptive_gripper.urdf (robot description, URDF)
Before this commit: robot firefighter, 15 links, 14 joints
Joints:
- joint gripper_left3_to_gripper_left1: mimic joint=gripper_controller multiplier=-1.0 offset=0 -> (none)
- joint gripper_right3_to_gripper_right1: mimic joint=gripper_controller multiplier=1.0 offset=0 -> (none)
